File: CANduino128.kicad_pcb (KiCad board)
At the start: 2 copper layers, 95.9 x 90.2 mm, 145 parts, among them J1 Conn_02x32_Row_Letter_First, J2 Conn_01x10, U1 AVR-H128-CAN, U2 74AHC373

Commit message: It's the fanal countdown tadadaaaada tadada ! Bon pour v3.1
git-svn-id: file:///D%5C00%20-%20Dev%20&%20Calculs%5CRepoTortoiseSVN_PCB%5CCANduino128/tags/CANduino128%20-%20v3.0@71 67ddf66f-3787-a644-8df7-7746e21a92b3
Parts:
- removed kibuzzard-6252E51C (x2): G***, kibuzzard-6252E51C
- removed kibuzzard-6252E525 (x2): G***, kibuzzard-6252E525
- removed kibuzzard-62533B1F: G***, kibuzzard-62533B1F
- removed kibuzzard-62533B3B: G***, kibuzzard-62533B3B
- removed kibuzzard-62533B4F: G***, kibuzzard-62533B4F
- removed kibuzzard-62533B5C: G***, kibuzzard-62533B5C
- removed kibuzzard-62533B6F: G***, kibuzzard-62533B6F
- removed kibuzzard-62533B79: G***, kibuzzard-62533B79
- removed kibuzzard-62533B82: G***, kibuzzard-62533B82
- removed kibuzzard-62E5227E: G***, kibuzzard-62E5227E
- removed kibuzzard-62E522CF: G***, kibuzzard-62E522CF
- removed kibuzzard-62F030DA: G***, kibuzzard-62F030DA
- removed kibuzzard-62F694D7: G***, kibuzzard-62F694D7
- removed kibuzzard-62F7C70C: G***, kibuzzard-62F7C70C
- removed kibuzzard-62F7C725: G***, kibuzzard-62F7C725
- removed kibuzzard-62F7C737: G***, kibuzzard-62F7C737
- removed kibuzzard-62F7C766: G***, kibuzzard-62F7C766
- added kibuzzard-638696BA: G***, kibuzzard-638696BA, F.Cu at (149.9, 130.2)
- added kibuzzard-638696BA: G***, kibuzzard-638696BA, F.Cu at (154.9, 130.2)
- added kibuzzard-638696E0: G***, kibuzzard-638696E0, F.Cu at (147.3, 130.2)
- added kibuzzard-638696E0: G***, kibuzzard-638696E0, F.Cu at (152.4, 130.2)
- added kibuzzard-63869728: G***, kibuzzard-63869728, F.Cu at (144.8, 130.2)
- added kibuzzard-63869737: G***, kibuzzard-63869737, F.Cu at (142.2, 130.2)
- added kibuzzard-63869742: G***, kibuzzard-63869742, F.Cu at (139.7, 130.2)
- added kibuzzard-6386974E: G***, kibuzzard-6386974E, F.Cu at (137.2, 130.2)
- kibuzzard-6383CA6D: moved to F.Cu
- moved kibuzzard-6383CA6D 73.7 mm to (125.7, 88.9)
- moved kibuzzard-62F6996F 12.0 mm to (174.0, 124.5), turned to -90 degrees
- moved kibuzzard-62533389 11.4 mm to (123.2, 59.7)
- moved kibuzzard-625333BD 11.4 mm to (123.2, 64.8)
- moved kibuzzard-625333D2 11.4 mm to (123.2, 69.8)
- moved kibuzzard-625333E4 11.4 mm to (123.2, 108.0)
- moved kibuzzard-625333EE 11.4 mm to (123.2, 113.0)
- moved kibuzzard-625333F8 11.4 mm to (123.2, 118.1)
- moved kibuzzard-62533490 11.4 mm to (123.2, 74.9)
- moved kibuzzard-625334E2 11.4 mm to (123.2, 97.8)
- moved kibuzzard-625334F4 11.4 mm to (123.2, 102.9)
- moved kibuzzard-627C3911 11.4 mm to (123.2, 92.7)
- moved kibuzzard-627C397B 11.4 mm to (123.2, 80.0)
- moved kibuzzard-627C3994 11.4 mm to (123.2, 85.1)
- moved kibuzzard-6252E636 10.2 mm to (111.8, 72.4)
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Routing:
- net ~{RESET}: track 83.8 -> 90.1 mm
- net T0_OC0x: track 122.0 -> 127.1 mm
- net GND: track 414.7 -> 418.4 mm
- net Net-(LED_D9-Pad2): track 82.7 -> 81.7 mm
- net DAI0: track 26.9 -> 26.1 mm
Other:
- outline, holes or cut-outs redrawn
- board text added: "GND A0 A1 A2 A3 A4 A5 A6 A7 A8 A9 A10 A11 A12 A13 A14 A15 GND GND GND GND +5V GND D0 D1 D2 D3 D4 D5 D6 D7 +5V"
- board text added: "GND DAI7 DAI6 DAI5 DAI4 DAI3 DAI2 DAI1 DAI0 ARef"
- board text added: "GND GND T0 +5V ALE GND +5V GND GND GND GND GND ICP1 +5V GND +5V GND +5V +5V +5V ~{RD} ~{WR} GND +Batt +5V x GND x GND +5V ~{RST} GND"
- board text removed: "T0-0C0x"

Commit message: Avec les réglages "Rancunes"
git-svn-id: file:///D%5C00%20-%20Dev%20&%20Calculs%5CRepoTortoiseSVN_PCB%5CCANduino128/tags/CANduino128%20-%20v3.0@73 67ddf66f-3787-a644-8df7-7746e21a92b3
Other:
- rule pad_to_mask_clearance: 0 -> 0.1
Changed lines of the file:
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@@
       (dielectric_constraints no)
     )
-    (pad_to_mask_clearance 0)
+    (pad_to_mask_clearance 0.1)
+    (pad_to_paste_clearance_ratio -0.1)
     (pcbplotparams
       (layerselection 0x00010fc_ffffffff)
@@
     )
     (fp_poly (pts
+        (xy -0.388144 -0.300038)
+        (xy -0.417513 -0.194469)
+        (xy -0.442913 -0.096044)
+        (xy -0.465138 0.001588)
+        (xy -0.484981 0.103188)
+        (xy -0.292894 0.103188)
+        (xy -0.311944 0.001588)
+        (xy -0.333375 -0.096044)
+        (xy -0.358775 -0.194469)
+        (xy -0.388144 -0.300038)
+      ) (layer "F.SilkS") (width 0) (fill solid))
+    (fp_poly (pts
         (xy -1.534319 -1.025393)
         (xy -1.408113 -0.378619)
@@
         (xy -1.534319 -1.025393)
       ) (layer "F.SilkS") (width 0) (fill solid))
-    (fp_poly (pts
-        (xy -0.388144 -0.300038)
-        (xy -0.417513 -0.194469)
-        (xy -0.442913 -0.096044)
-        (xy -0.465138 0.001588)
-        (xy -0.484981 0.103188)
-        (xy -0.292894 0.103188)
-        (xy -0.311944 0.001588)
-        (xy -0.333375 -0.096044)
-        (xy -0.358775 -0.194469)
-        (xy -0.388144 -0.300038)
-      ) (layer "F.SilkS") (width 0) (fill solid))
   )
