File: CANduino128.kicad_pcb (KiCad board)
At the start: 2 copper layers, 95.9 x 90.2 mm, 130 parts, among them J1 Conn_01x02, J2 Conn_01x10, J3 AVR-USBASP-target, U1 AVR-H128-CAN, U2 74AHC373, U3 4555

Commit message: On se cherche encore sur les /CS qui vont sur les DRQx ou les /DRAQx
git-svn-id: file:///D%5C00%20-%20Dev%20&%20Calculs%5CRepoTortoiseSVN_PCB%5CCANduino128/branches/CANduino128%20-%20v3.x@99 67ddf66f-3787-a644-8df7-7746e21a92b3
Parts:
- J3: footprint Connector_PinHeader_2.54mm:PinHeader_2x05_P2.54mm_Vertical -> Connector_IDC:IDC-Header_2x05_P2.54mm_Vertical
- kibuzzard-62F83662: moved to B.Cu
- moved LED_D9 36.7 mm to (111.8, 111.8), turned to 90 degrees
- moved R_LED_D9 29.3 mm to (111.8, 105.4), turned to -90 degrees
- moved kibuzzard-6252E5C3 27.3 mm to (111.8, 98.4)
- moved CAN_RX_1 6.35 mm to (111.8, 118.1)
- moved kibuzzard-62F83662 5.71 mm to (111.8, 112.4)
Routing:
- net GND: track 761.7 -> 793.0 mm
- net +BATT: track 132.4 -> 160.0 mm
- net SCK_LED_D9: track 48.7 -> 60.7 mm
- net CAN_RX: track 122.8 -> 116.9 mm
- net /ADR7-D7: track 72.3 -> 74.5 mm
- net RXD_PDI: track 28.4 -> 29.5 mm
- net /ADR7: track 47.2 -> 48.1 mm
- net TXD_PDO: track 30.9 -> 31.7 mm

Commit message: Last version pour la v3.2 On arrête les frais sur cette carte
git-svn-id: file:///D%5C00%20-%20Dev%20&%20Calculs%5CRepoTortoiseSVN_PCB%5CCANduino128/branches/CANduino128%20-%20v3.x@100 67ddf66f-3787-a644-8df7-7746e21a92b3
Parts:
- removed C_4555: 100nF, Capacitor_SMD:C_1210_3225Metric_Pad1.33x2.70mm_HandSolder
- removed RST1: MountingHole_Pad, Connector_Wire:SolderWire-0.1sqmm_1x01_D0.4mm_OD1mm
- removed U3: 4555, Package_DIP_AKL:DIP-16_W7.62mm_Socket
- removed kibuzzard-62F7E6CE: G***, kibuzzard-62F7E6CE
- removed kibuzzard-62F834DA: G***, kibuzzard-62F834DA
- Pad_SCL1, Pad_SDA1: footprint Jumper:SolderJumper-2_P1.3mm_Open_TrianglePad1.0x1.5mm -> Connector_PinHeader_2.54mm:PinHeader_1x02_P2.54mm_Vertical
- moved Pad_SCL1 20.5 mm to (139.7, 88.9), turned to 0 degrees
- moved Pad_SDA1 20.5 mm to (144.8, 88.9), turned to 0 degrees
- moved R_SCL1 20.2 mm to (139.7, 84.1)
- moved R_SDA1 20.2 mm to (144.8, 84.1)
- moved RS_K10 17.3 mm to (142.9, 106.0), turned to 0 degrees
- moved C_2551 10.8 mm to (162.6, 104.1), turned to 90 degrees
- moved MCP1 6.83 mm to (157.5, 107.9), turned to 180 degrees
- moved kibuzzard-627FBB38 5.08 mm to (125.1, 83.8)
- moved kibuzzard-638696BA 5.08 mm to (125.1, 88.9)
- moved kibuzzard-627FBB28 5.08 mm to (125.1, 81.3)
- moved kibuzzard-638696E0 5.08 mm to (125.1, 86.4)
- moved J3 1.27 mm to (115.6, 62.2)
Connections:
- BusISA8 pad 16: DRQ3 -> unconnected-(BusISA8-DRQ3-Pad16)
- BusISA8 pad 18: DRQ1 -> unconnected-(BusISA8-DRQ1-Pad18)
- BusISA8 pad 20: unconnected-(BusISA8-BCLK-Pad20) -> SysClk
- BusISA8 pad 30: unconnected-(BusISA8-OSC-Pad30) -> /ADR15
- BusISA8 pad 44: unconnected-(BusISA8-BA19-Pad44) -> ~{CS3}
- BusISA8 pad 6: DRQ2 -> unconnected-(BusISA8-DRQ2-Pad6)
- J3 pad 4: RXD_PDI -> unconnected-(J3-RXD_target-Pad4)
- J3 pad 6: TXD_PDO -> unconnected-(J3-TXD_target-Pad6)
- J_Comm_0 pad 5: SCL_INT0 -> CANL
- J_Comm_0 pad 6: SDA_INT1 -> CANH
- J_Comm_0 pad 7: CANL -> SCL_INT0
- J_Comm_0 pad 8: CANH -> SDA_INT1
- U1 pad 14: ~{CS2} -> SysClk
Routing:
- net SysClk: track 0.00 -> 114.2 mm
- net DRQ2: track 80.7 -> 0.00 mm, vias 1 -> 0
- net DRQ1: track 53.7 -> 0.00 mm, vias 1 -> 0
- net GND: track 793.0 -> 843.5 mm
- net DRQ3: track 46.9 -> 0.00 mm, vias 1 -> 0
- net /ADR15: track 20.1 -> 56.7 mm
- net ~{CS2}: track 35.1 -> 0.00 mm
- net +5V: track 302.0 -> 277.1 mm, vias 1 -> 3
- net ~{CS3}: track 57.2 -> 38.5 mm
- net +BATT: track 160.0 -> 141.4 mm, vias 3 -> 1
- net SDA_INT1: track 83.0 -> 65.1 mm
- net CANH: track 64.3 -> 47.6 mm
- net SCL_INT0: track 79.4 -> 65.3 mm
- net CAN_RX: track 116.9 -> 103.6 mm
- net TXD_PDO: track 31.7 -> 21.4 mm
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Other:
- board text added: "CLK"
- board text added: "GND A0 A1 A2 A3 A4 A5 A6 A7 A8 A9 A10 A11 A12 A13 A14 A15 x x x ~{CS3} x x D0 D1 D2 D3 D4 D5 D6 D7 x"
- board text added: "GND GND X1 +5V ALE x x x x x x x OC2A x x x x x x x ~{RD} ~{WR} x +VIN x x x x x +5V ~{RST} GND"
- board text added: "OC2A"
- board text added: "~{CS3}"
- board text removed: "GND A0 A1 A2 A3 A4 A5 A6 A7 A8 A9 A10 A11 A12 A13 A14 A15 x x x x x x D0 D1 D2 D3 D4 D5 D6 D7 x"
- board text removed: "GND GND X1 +5V ALE x x x x x x x BCLK x x x x x x x ~{RD} ~{WR} x +VIN x x x x x +5V ~{RST} GND"
- board text removed: "RXD"
- board text removed: "TXD"
- board text removed: "USBAsp"
