File: CANduino128.kicad_pcb (KiCad board)
At the start: 2 copper layers, 95.9 x 90.2 mm, 78 parts, among them J1 Conn_02x14_Odd_Even, J2 Conn_01x10

Commit message: [UPGRADE] : Changement de bus interne de communication (pas de rétrocompatibilité) - remplacement du connecteur double par un seul connecteur IDE 40pin - rerouting léger
Parts:
- removed PCIe_CAN_1: Conn_02x07_Odd_Even, Connector_PinHeader_2.54mm:PinHeader_2x07_P2.54mm_Vertical
- removed PCIe_SPI_1: Conn_02x11_Odd_Even, Connector_PinHeader_2.54mm:PinHeader_2x11_P2.54mm_Vertical
- removed kibuzzard-6252DD85: G***, kibuzzard-6252DD85
- removed kibuzzard-6252DDA8: G***, kibuzzard-6252DDA8
- added J3: Conn_02x20_Odd_Even, Connector_IDC:IDC-Header_2x20_P2.54mm_Vertical, F.Cu at (109.2, 113.0)
- moved RST1 7.65 mm to (114.3, 83.8)
- moved LED_RX1 4.02 mm to (121.9, 120.7)
- moved LED_TX1 4.02 mm to (121.9, 116.8)
- moved kibuzzard-62799BC1 2.62 mm to (107.3, 57.1)
- moved Pad_R1 1.27 mm to (115.6, 61.0)
Routing:
- net GND: track 539.3 -> 900.4 mm
- net CAN_RX: track 70.7 -> 65.4 mm
- net Net-(LED_RX1-A): track 33.3 -> 30.6 mm
- net ~{RESET}: track 27.9 -> 25.1 mm
- net SCK_LED_D9: track 76.9 -> 79.3 mm
- net CIPO: track 61.0 -> 63.0 mm
- net +BATT: track 110.5 -> 108.7 mm
- net COPI: track 60.9 -> 62.5 mm
- net Net-(Pad_R1-B): track 4.80 -> 6.07 mm
- net /ADR15: track 117.8 -> 116.5 mm
- net ~{CS}: track 65.7 -> 67.0 mm
- net /~{SPI_CS2}: track 34.1 -> 33.2 mm
- net +5V: track 319.7 -> 320.2 mm
- net SCL_INT0: track 41.5 -> 42.0 mm
- net SDA_INT1: track 46.5 -> 46.0 mm
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Other:
- board text added: "CANH"
- board text added: "CANL"
- board text added: "LED RX"
- board text added: "LED TX"
- board text added: "MBusA"
- board text added: "MBusB"
- board text removed: "CAN0H"
- board text removed: "CAN0L"
- board text removed: "CAN1H"
- board text removed: "CAN1L"

Commit message: [UPGRADE] : OC2A sur OSC1 + suppression des vias
Parts:
- moved R_TX_1 32.0 mm to (115.6, 120.7), turned to 0 degrees
- moved R_RX_1 31.5 mm to (115.6, 116.2), turned to 0 degrees
- moved R_SCL1 24.3 mm to (135.9, 97.8), turned to 90 degrees
- moved Pad_SCL1 23.6 mm to (135.9, 102.2)
- moved Pad_SDA1 23.5 mm to (139.7, 102.2)
- moved R_SDA1 17.9 mm to (139.7, 97.8), turned to 90 degrees
- moved LED_RX1 4.45 mm to (121.9, 116.2), turned to 180 degrees
- moved LED_TX1 3.81 mm to (121.9, 120.7), turned to 180 degrees
Connections:
- AT90CAN128 pad 14: /~{SPI_CS3} -> /SWClk
- J3 pad 21: /~{SPI_CS3} -> /Connection PCI CAN Express/UPDI
- J3 pad 30: /Connection PCI CAN Express/OSC1 -> /SWClk
Routing:
- net /SWClk: track 0.00 -> 93.3 mm
- net GND: track 900.4 -> 810.8 mm, vias 1 -> 0
- net ~{RESET}: track 25.1 -> 96.9 mm, vias 1 -> 0
- net /~{SPI_CS3}: track 40.7 -> 0.00 mm, vias 1 -> 0
- net CANH: track 55.8 -> 96.0 mm, vias 1 -> 0
- net CANL: track 54.1 -> 83.6 mm, vias 1 -> 0
- net Net-(LED_RX1-A): track 30.6 -> 3.31 mm
- net Net-(LED_TX1-A): track 26.8 -> 3.31 mm
- net +5V: track 320.2 -> 337.1 mm, vias 3 -> 0
- net ~{WR}-D26: track 26.7 -> 12.7 mm
- net +BATT: track 108.7 -> 120.6 mm
- net CAN_TX: track 35.6 -> 46.5 mm
- net /~{SPI_CS2}: track 33.2 -> 43.0 mm, vias 1 -> 0
- net Net-(Pad_SDA1-A): track 8.06 -> 2.17 mm
- net CAN_RX: track 65.4 -> 71.0 mm
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Other:
- board text removed: "LED RX"
- board text removed: "LED TX"
