File: CANduino128.kicad_sch (KiCad schematic)
At the start: 62 parts, among them J1 Conn_02x14_Odd_Even, J2 Conn_01x10

Commit message: git-svn-id: file:///D%5C00%20-%20Dev%20&%20Calculs%5CRepoTortoiseSVN_PCB%5CCANduino128/branches/CANduino128%20-%20v3.1a@64 67ddf66f-3787-a644-8df7-7746e21a92b3
Parts:
- removed D25: MountingHole_Pad, Connector_Wire:SolderWire-0.5sqmm_1x01_D0.9mm_OD2.1mm, symbol Mechanical:MountingHole_Pad
Connections:
- net T0_OC0x is gone; now on net ~{SPI_CS2}: AT90CAN128.32 (PD7-D25)
- net ADR0: now also 74AHC373.19 (O7); no longer 74AHC373.2 (O0)
- net ADR0-D0: now also 74AHC373.18 (D7); no longer 74AHC373.3 (D0)
- net ADR1: now also 74AHC373.2 (O0); no longer 74AHC373.19 (O7)
- net ADR1-D1: now also 74AHC373.3 (D0); no longer 74AHC373.18 (D7)
- net ADR2: now also 74AHC373.16 (O6); no longer 74AHC373.5 (O1)
- net ADR2-D2: now also 74AHC373.17 (D6); no longer 74AHC373.4 (D1)
- net ADR3: now also 74AHC373.5 (O1); no longer 74AHC373.16 (O6)
- net ADR3-D3: now also 74AHC373.4 (D1); no longer 74AHC373.17 (D6)
- net ADR4: now also 74AHC373.15 (O5); no longer 74AHC373.6 (O2)
- net ADR4-D4: now also 74AHC373.14 (D5); no longer 74AHC373.7 (D2)
- net ADR5: now also 74AHC373.9 (O3); no longer 74AHC373.15 (O5)
- net ADR5-D5: now also 74AHC373.8 (D3); no longer 74AHC373.14 (D5)
- net ADR6: now also 74AHC373.12 (O4); no longer 74AHC373.9 (O3)
- net ADR6-D6: now also 74AHC373.13 (D4); no longer 74AHC373.8 (D3)
- net ADR7: now also 74AHC373.6 (O2); no longer 74AHC373.12 (O4)
- net ADR7-D7: now also 74AHC373.7 (D2); no longer 74AHC373.13 (D4)
- net DAI0: now also AT90CAN128.61 (ADC0-A0/D45-PF0); no longer J2.9 (Pin_9)
- net DAI1: now also AT90CAN128.60 (ADC1-A1/D46-PF1); no longer J2.8 (Pin_8)
- net DAI2: now also AT90CAN128.59 (ADC2-A2/D47-PF2); no longer J2.7 (Pin_7)
- net DAI3: now also AT90CAN128.58 (ADC3-A3/D48-PF3); no longer J2.6 (Pin_6)
- net DAI4: now also AT90CAN128.57 (ADC4-A4/D49-PF4); no longer J2.5 (Pin_5)
- net DAI5: now also AT90CAN128.56 (ADC5-A5/D50-PF5); no longer J2.4 (Pin_4)
- net DAI6: now also AT90CAN128.55 (ADC6-A6/D51-PF6); no longer J2.3 (Pin_3)
- net DAI7: now also AT90CAN128.54 (ADC7-A7/D52-PF7); no longer J2.2 (Pin_2)
- net GP0: now also J2.9 (Pin_9); no longer AT90CAN128.61 (ADC0-A0/D45-PF0)
- net GP1: now also J2.8 (Pin_8); no longer AT90CAN128.60 (ADC1-A1/D46-PF1)
- net GP2: now also J2.7 (Pin_7); no longer AT90CAN128.59 (ADC2-A2/D47-PF2)
- net GP3: now also J2.6 (Pin_6); no longer AT90CAN128.58 (ADC3-A3/D48-PF3)
- net GP4: now also J2.5 (Pin_5); no longer AT90CAN128.57 (ADC4-A4/D49-PF4)
- net GP5: now also J2.4 (Pin_4); no longer AT90CAN128.56 (ADC5-A5/D50-PF5)
- net GP6: now also J2.3 (Pin_3); no longer AT90CAN128.55 (ADC6-A6/D51-PF6)
- net GP7: now also J2.2 (Pin_2); no longer AT90CAN128.54 (ADC7-A7/D52-PF7)
- no-connect marks 10 -> 9

Commit message: git-svn-id: file:///D%5C00%20-%20Dev%20&%20Calculs%5CRepoTortoiseSVN_PCB%5CCANduino128/branches/CANduino128%20-%20v3.1a@65 67ddf66f-3787-a644-8df7-7746e21a92b3
Parts:
- removed CA1, CA2, CA3, CA4, CA5, CA6, CA7, CA8: 1000pF, Capacitor_SMD:C_1210_3225Metric_Pad1.33x2.70mm_HandSolder, symbol Device:C_Small
- removed JPA1, JPA2, JPA3, JPA4, JPA5, JPA6, JPA7, JPA8: SolderJumper_2_Open, Jumper:SolderJumper-2_P1.3mm_Open_TrianglePad1.0x1.5mm, symbol Jumper:SolderJumper_2_Open
- removed R1_A1, R1_A2, R1_A3, R1_A4, R1_A5, R1_A6, R1_A7, R1_A8: 1K, Resistor_SMD:R_1210_3225Metric_Pad1.30x2.65mm_HandSolder, symbol Device:R_Small
- added H7, H8: MountingHole_Pad, Connector_Wire:SolderWire-0.1sqmm_1x01_D0.4mm_OD1mm, symbol Mechanical:MountingHole_Pad
Connections:
- net +BATT: now also H7.1
- net GND: now also H8.1
Other:
- added sheet ADC_Line0 (ADC_Line.kicad_sch)
- added sheet ADC_Line1 (ADC_Line.kicad_sch)
- added sheet ADC_Line2 (ADC_Line.kicad_sch)
- added sheet ADC_Line3 (ADC_Line.kicad_sch)
- added sheet ADC_Line4 (ADC_Line.kicad_sch)
- added sheet ADC_Line5 (ADC_Line.kicad_sch)
- added sheet ADC_Line6 (ADC_Line.kicad_sch)
- added sheet ADC_Line7 (ADC_Line.kicad_sch)
- moved on the sheet: J2, PCIe_CAN_1, PCIe_SPI_1

Commit message: Houlà ! On y est presque ! Un peu de silkscreen à mettre à jour et on aura une révision livrable.
git-svn-id: file:///D%5C00%20-%20Dev%20&%20Calculs%5CRepoTortoiseSVN_PCB%5CCANduino128/branches/CANduino128%20-%20v3.1a@66 67ddf66f-3787-a644-8df7-7746e21a92b3
Parts:
- removed H5, H6: MountingHole_Pad, Connector_Wire:SolderWire-0.1sqmm_1x01_D0.4mm_OD1mm_Relief2x, symbol Mechanical:MountingHole_Pad
- removed H7, H8: MountingHole_Pad, Connector_Wire:SolderWire-0.1sqmm_1x01_D0.4mm_OD1mm, symbol Mechanical:MountingHole_Pad
- added J_Batt_Int0, J_Batt_Strap0: Conn_01x02, Connector_PinHeader_2.54mm:PinHeader_1x02_P2.54mm_Vertical, symbol Connector_Generic:Conn_01x02
- added J_Batt_PPal0: Conn_01x02, TerminalBlock_TE-Connectivity:TerminalBlock_TE_282834-2_1x02_P2.54mm_Horizontal, symbol Connector_Generic:Conn_01x02
- added Trou_Alim_0: MountingHole_Pad, MountingHole:MountingHole_4.3mm_M4_ISO14580_Pad, symbol Mechanical:MountingHole_Pad
Connections:
- net +BATT: now also J_Batt_Int0.1 (Pin_1), J_Batt_PPal0.1 (Pin_1), J_Batt_Strap0.1 (Pin_1)
- net GND: now also J_Batt_Int0.2 (Pin_2), J_Batt_PPal0.2 (Pin_2), J_Batt_Strap0.2 (Pin_2), Trou_Alim_0.1

Commit message: Silkscreen terminé. Bon pour release après une dernière vérif.
git-svn-id: file:///D%5C00%20-%20Dev%20&%20Calculs%5CRepoTortoiseSVN_PCB%5CCANduino128/branches/CANduino128%20-%20v4.0a@70 67ddf66f-3787-a644-8df7-7746e21a92b3
Parts:
- removed J_Batt_Int0, J_Batt_Strap0: Conn_01x02, Connector_PinHeader_2.54mm:PinHeader_1x02_P2.54mm_Vertical, symbol Connector_Generic:Conn_01x02
- removed Trou_Alim_0: MountingHole_Pad, MountingHole:MountingHole_4.3mm_M4_ISO14580_Pad, symbol Mechanical:MountingHole_Pad
Other:
- moved on the sheet: J1, J_Batt_PPal0, KiCad0, LED_D9, LED_PWR5, LED_RX1, LED_TX1, PCIe_CAN_1, PCIe_SPI_1, R_LED_D9, R_LED_PWR1, R_RX_1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

Commit message: KiCad 7.0 SPI_CS3 Reste simplification du chemin Redondance alim +5V
Mais surtout KiCad 7.0 qui empêche la rétrocompatibilité avec les version antérieure sous KiCad 6.x

git-svn-id: file:///D%5C00%20-%20Dev%20&%20Calculs%5CRepoTortoiseSVN_PCB%5CCANduino128/branches/CANduino128%20-%20v4.0a@84 67ddf66f-3787-a644-8df7-7746e21a92b3
Parts:
- MCP2551: footprint Package_DIP:DIP-8_W7.62mm -> Package_DIP:DIP-8_W7.62mm_Socket
Connections:
- net SysClk is gone; now on net ~{SPI_CS3}: AT90CAN128.14 (PB4-D12-OC2A)
- no-connect marks 9 -> 7
Other:
- note added: "(SysClk)"
