File: DemuxDRQx.kicad_sch (KiCad schematic)
At the start: 1 part, among them U3 4555

Commit message: Déplacement des connecteurs BLDC Reroute Ajout d'un connecteur ICSP de type USBAsp
git-svn-id: file:///D%5C00%20-%20Dev%20&%20Calculs%5CRepoTortoiseSVN_PCB%5CCANduino128/branches/CANduino128%20-%20v3.x@98 67ddf66f-3787-a644-8df7-7746e21a92b3
Parts:
- U3: footprint Package_DIP_AKL:DIP-16_W7.62mm_Socket_LongPads -> Package_DIP_AKL:DIP-16_W7.62mm_Socket
Changed lines of the file:
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@@
       (effects (font (size 1.27 1.27)) (justify left))
     )
-    (property "Footprint" "Package_DIP_AKL:DIP-16_W7.62mm_Socket_LongPads" (at 120.65 135.89 0)
+    (property "Footprint" "Package_DIP_AKL:DIP-16_W7.62mm_Socket" (at 120.65 135.89 0)
       (effects (font (size 1.27 1.27)) hide)
     )
@@
       (effects (font (size 1.27 1.27)) (justify left))
     )
-    (property "Footprint" "Package_DIP_AKL:DIP-16_W7.62mm_Socket_LongPads" (at 120.65 99.06 0)
+    (property "Footprint" "Package_DIP_AKL:DIP-16_W7.62mm_Socket" (at 120.65 99.06 0)
       (effects (font (size 1.27 1.27)) hide)
     )

Commit message: On se cherche encore sur les /CS qui vont sur les DRQx ou les /DRAQx
git-svn-id: file:///D%5C00%20-%20Dev%20&%20Calculs%5CRepoTortoiseSVN_PCB%5CCANduino128/branches/CANduino128%20-%20v3.x@99 67ddf66f-3787-a644-8df7-7746e21a92b3
Parts:
- removed U3: 4555, Package_DIP_AKL:DIP-16_W7.62mm_Socket, symbol 4xxx_IEEE:4555
- added U4: 4556, symbol 4xxx_IEEE:4556
Connections:
- net VIN: now also U4.16 (Vdd), U4.16 (Vdd)
- net VSS: now also U4.1 (~{EN}), U4.8 (Vss), U4.8 (Vss)
- net ~{CS_A0}: now also U4.2 (A0)
- net ~{CS_A1}: now also U4.3 (A1)
- new net ~{DRQ1}: U4.6 (~{Q2})
- new net ~{DRQ2}: U4.5 (~{Q1})
- new net ~{DRQ3}: U4.4 (~{Q0})
Other:
- note added: "D3 D2 D1 nc B A | Q0 Q1 Q2 Q3 ----|------------ 0 0 | 0 1 1 1 0 1 | 1 0 1 1 1 0 | 1 1 0 1 1 1 | 1 1 1 0"
- note removed: "D3 D2 D1 nc B A | Q0 Q1 Q2 Q3 ----|------------ 0 0 | 1 0 0 0 0 1 | 0 1 0 0 1 0 | 0 0 1 0 1 1 | 0 0 0 1"
Changed lines of the file:
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@@
     (stroke (width 0) (type default))
   )
-  (text "      D3 D2 D1 nc\nB A | Q0 Q1 Q2 Q3\n----|------------\n0 0 | 1  0  0  0\n0 1 | 0  1  0  0\n1 0 | 0  0  1  0\n1 1 | 0  0  0  1"
+  (text "      D3 D2 D1 nc\nB A | Q0 Q1 Q2 Q3\n----|------------\n0 0 | 0  1  1  1\n0 1 | 1  0  1  1\n1 0 | 1  1  0  1\n1 1 | 1  1  1  0"
     (at 140.97 119.38 0)
     (effects (font (face "Fira Code") (size 1.27 1.27)) (justify left bottom))
   )
-  (hierarchical_label "DRQ1" (shape output) (at 130.81 100.33 0) (fields_autoplaced)
+  (hierarchical_label "~{DRQ1}" (shape output) (at 130.81 100.33 0) (fields_autoplaced)
     (effects (font (size 1.27 1.27)) (justify left))
   )
@@
     (effects (font (size 1.27 1.27)) (justify right))
   )
-  (hierarchical_label "DRQ2" (shape output) (at 130.81 97.79 0) (fields_autoplaced)
+  (hierarchical_label "~{DRQ2}" (shape output) (at 130.81 97.79 0) (fields_autoplaced)
     (effects (font (size 1.27 1.27)) (justify left))
   )
@@
     (effects (font (size 1.27 1.27)) (justify left))
   )
-  (hierarchical_label "DRQ3" (shape output) (at 130.81 95.25 0) (fields_autoplaced)
+  (hierarchical_label "~{DRQ3}" (shape output) (at 130.81 95.25 0) (fields_autoplaced)
     (effects (font (size 1.27 1.27)) (justify left))
   )
@@
     (effects (font (size 1.27 1.27)) (justify left))
   )
-  (symbol (lib_id "4xxx_IEEE:4555") (at 120.65 135.89 0) (unit 1)
+  (symbol (lib_id "4xxx_IEEE:4556") (at 120.65 135.89 0) (unit 2)
     (in_bom yes) (on_board yes) (dnp no) (fields_autoplaced)
-    (property "Reference" "U3" (at 122.8441 124.46 0)
+    (property "Reference" "U4" (at 122.8441 124.46 0)
       (effects (font (size 1.27 1.27)) (justify left))
     )
-    (property "Value" "4555" (at 122.8441 127 0)
+    (property "Value" "4556" (at 122.8441 127 0)
       (effects (font (size 1.27 1.27)) (justify left))
     )
-    (property "Footprint" "Package_DIP_AKL:DIP-16_W7.62mm_Socket" (at 120.65 135.89 0)
+    (property "Footprint" "" (at 120.65 135.89 0)
       (effects (font (size 1.27 1.27)) hide)
     )
-    (property "Datasheet" "https://datasheet.lcsc.com/lcsc/2302221530_Texas-Instruments-CD4556BE_C1547267.pdf" (at 120.65 135.89 0)
+    (property "Datasheet" "" (at 120.65 135.89 0)
       (effects (font (size 1.27 1.27)) hide)
     )
@@
     (instances
       (project "CANduino128"
-        (path "/b26d10c1-0874-459a-80a4-e525262e670c"
-          (reference "U3") (unit 1)
-        )
         (path "/b26d10c1-0874-459a-80a4-e525262e670c/359473b5-ba41-473b-8aac-b24c5eb2401e"
-          (reference "U3") (unit 1)
+          (reference "U4") (unit 2)
         )
       )
     )
   )
-  (symbol (lib_id "4xxx_IEEE:4555") (at 120.65 99.06 0) (unit 2)
+  (symbol (lib_id "4xxx_IEEE:4556") (at 120.65 99.06 0) (unit 1)
     (in_bom yes) (on_board yes) (dnp no) (fields_autoplaced)
-    (property "Reference" "U3" (at 122.8441 87.63 0)
+    (property "Reference" "U4" (at 122.8441 87.63 0)
       (effects (font (size 1.27 1.27)) (justify left))
     )
-    (property "Value" "4555" (at 122.8441 90.17 0)
+    (property "Value" "4556" (at 122.8441 90.17 0)
       (effects (font (size 1.27 1.27)) (justify left))
     )
-    (property "Footprint" "Package_DIP_AKL:DIP-16_W7.62mm_Socket" (at 120.65 99.06 0)
+    (property "Footprint" "" (at 120.65 99.06 0)
       (effects (font (size 1.27 1.27)) hide)
     )
-    (property "Datasheet" "https://datasheet.lcsc.com/lcsc/2302221530_Texas-Instruments-CD4556BE_C1547267.pdf" (at 120.65 99.06 0)
+    (property "Datasheet" "" (at 120.65 99.06 0)
       (effects (font (size 1.27 1.27)) hide)
     )
@@
     (instances
       (project "CANduino128"
-        (path "/b26d10c1-0874-459a-80a4-e525262e670c"
-          (reference "U3") (unit 2)
-        )
         (path "/b26d10c1-0874-459a-80a4-e525262e670c/359473b5-ba41-473b-8aac-b24c5eb2401e"
-          (reference "U3") (unit 2)
+          (reference "U4") (unit 1)
         )
       )
